File: mcu.kicad_sch (KiCad schematic)
At the start: 18 parts, among them IC1 STM32L051C6T6, J1 Conn_01x05_Pin, J2 Conn_01x03_Pin, SW1 PTS 647 SN50 SMTR2 LFS, Y1 8MHz, Y2 32.768KHZ

Commit message: added MOSFET, and switch for Servos
Parts:
- SW1: footprint ExpansionBoardFootprints:Expansion Button PTS 647 SN50 SMTR2 LFS -> AquaPartsLib:SW_PTS_647_SN50_SMTR2_LFS
Changed lines of the file:
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@@
 			)
 		)
-		(property "Footprint" "ExpansionBoardFootprints:Expansion Button PTS 647 SN50 SMTR2 LFS"
+		(property "Footprint" "AquaPartsLib:SW_PTS_647_SN50_SMTR2_LFS"
 			(at 118.11 156.21 0)
 			(effects
